File: r4s_flash.kicad_pcb (KiCad board)
At the start: 2 copper layers, 19.5 x 14.5 mm, 8 parts, among them J1 NanoPi_R4S_Header, SW1 SW_DIP_x02, U1 SST25VF080B-50-4x-S2Ax, U2 M24C02-WMN

Commit message: Add rev1.1
Parts:
- removed R3: 10k, Resistor_SMD:R_0805_2012Metric_Pad1.20x1.40mm_HandSolder
- removed U2: M24C02-WMN, Package_SO:SOIC-8_3.9x4.9mm_P1.27mm
- C1: footprint Capacitor_SMD:C_0603_1608Metric_Pad1.08x0.95mm_HandSolder -> Capacitor_SMD:C_0805_2012Metric_Pad1.18x1.45mm_HandSolder; moved to F.Cu
- R1, R2: moved to F.Cu
- moved R1 13.1 mm to (157.5, 105.5), turned to 0 degrees
- moved R2 10.0 mm to (157.5, 103.2), turned to 0 degrees
- moved SW1 7.85 mm to (157.1, 98.1), turned to 90 degrees
- moved U1 3.78 mm to (151.6, 98.7), turned to -90 degrees
- moved C1 1.33 mm to (152.2, 104.8)
Connections:
- J1 pad 4: /I2C3_SDA -> unconnected-(J1-Pin_4-Pad4)
- J1 pad 6: /I2C3_SCL -> unconnected-(J1-Pin_6-Pad6)
- SW1 pad 1: /EEPROM_WP -> /FLASH_HOLD
- SW1 pad 4: +3.3V -> GND
Routing:
- net +3.3V: track 39.9 -> 15.8 mm, vias 3 -> 0
- net /I2C3_SCL: track 11.5 -> 0.00 mm
- net /EEPROM_WP: track 9.39 -> 0.00 mm, vias 1 -> 0
- net /I2C3_SDA: track 8.11 -> 0.00 mm
- net /FLASH_WP: track 7.24 -> 13.4 mm, vias 1 -> 2
- net /SPI1_TXD: track 11.9 -> 5.80 mm, vias 2 -> 0
- net /SPI1_CLK: track 20.5 -> 14.8 mm, vias 2 -> 0
- net /SPI1_RXD: track 3.23 -> 8.06 mm
- net /SPI1_CSn: track 9.58 -> 14.1 mm
- net /FLASH_HOLD: track 8.16 -> 10.7 mm, vias 1 -> 0
- net GND: track 0.45 -> 0.00 mm, vias 5 -> 6
Other:
- board size 19.5 x 14.5 mm -> 19.8 x 14.5 mm
- board text added: "H"
- board text added: "P"
- board text added: "Rev 1.1"
- board text removed: "1: EEPROM 2: FLASH"
