File: r4s_flash.kicad_sch (KiCad schematic)
At the start: 8 parts, among them J1 NanoPi_R4S_Header, SW1 SW_DIP_x02, U1 SST25VF080B-50-4x-S2Ax, U2 M24C02-WMN

Commit message: Add rev1.1
Parts:
- removed R3: 10k, Resistor_SMD:R_0805_2012Metric_Pad1.20x1.40mm_HandSolder, symbol Device:R
- removed U2: M24C02-WMN, Package_SO:SOIC-8_3.9x4.9mm_P1.27mm, symbol Memory_EEPROM:M24C02-WMN
- C1: footprint Capacitor_SMD:C_0603_1608Metric_Pad1.08x0.95mm_HandSolder -> Capacitor_SMD:C_0805_2012Metric_Pad1.18x1.45mm_HandSolder
Connections:
- net EEPROM_WP is gone; now on net FLASH_HOLD: SW1.1
- net +3.3V: no longer SW1.4
- net GND: now also SW1.4
- net I2C3_SCL: no longer names the net of J1.6 (Pin_6)
- net I2C3_SDA: no longer names the net of J1.4 (Pin_4)
Other:
- note removed: "i2c EEPROM"
- moved on the sheet: R1, R2, U1
